File: kicad/rf_bridge.kicad_pcb (KiCad board)
At the start: 2 copper layers, 25.4 x 45.7 mm, 16 parts, among them P1 CONN_01X08, P2 RF_TX, P3 RF_RX1, P4 RF_RX2, P5 BNC, U1 SA630

Commit message: pcb: A few tweaks for next version
Changed the footprint of the 10nF's to 0603, as I've discovered I have a
bout 1Kg of them.
Also changed pinout! Silly me, I used A6 and A7 pins on the arduidiot,
but these are ADC only, no digital logic. So luckily I had hooked up two
'spare' pins, so I switched to these instead.

Also, the rest of the PCB has beem tested, and the switch is defaulting
to the RX mode when EN pin is low (as expected), so the pulldown works
fine, and the AVR can keep it's antenna switch pin as open drain.

Signed-off-by: Michel Pollet <buserror@gmail.com>
Parts:
- C1, C2, C3, C4: footprint Capacitors_SMD:C_0805 -> Capacitors_SMD:C_0603
- R1: value 1K -> 10K
- moved R1 0.63 mm to (135.3, 102.9)
- moved C7 0.52 mm to (132.7, 89.5)
- moved C4 0.27 mm to (130.2, 89.5)
Connections:
- P1 pad 5: TX -> Net-(P1-Pad5)
- P1 pad 7: Net-(P1-Pad7) -> TX
- R2 pad 2: Net-(P1-Pad4) -> Net-(P1-Pad8)
Routing:
- net Net-(P1-Pad8): track 0.00 -> 24.9 mm, vias 0 -> 1
- net Net-(P1-Pad4): track 19.4 -> 0.15 mm, vias 1 -> 0
- net TX: track 17.1 -> 23.3 mm
- net Net-(C7-Pad1): track 3.07 -> 3.59 mm
- net Net-(C4-Pad1): track 2.54 -> 3.06 mm
Other:
- board text added: "rf_bridge 1.1"
- board text removed: "rf_bridge 1.0"
