File: kicad/rf_bridge.sch (KiCad schematic (older format))
At the start: 16 parts, among them P1 CONN_01X08, P2 RF_TX, P3 RF_RX1, P4 RF_RX2, P5 BNC, U1 SA630

Commit message: pcb: A few tweaks for next version
Changed the footprint of the 10nF's to 0603, as I've discovered I have a
bout 1Kg of them.
Also changed pinout! Silly me, I used A6 and A7 pins on the arduidiot,
but these are ADC only, no digital logic. So luckily I had hooked up two
'spare' pins, so I switched to these instead.

Also, the rest of the PCB has beem tested, and the switch is defaulting
to the RX mode when EN pin is low (as expected), so the pulldown works
fine, and the AVR can keep it's antenna switch pin as open drain.

Signed-off-by: Michel Pollet <buserror@gmail.com>
Parts:
- C1, C2, C3, C4: footprint Capacitors_SMD:C_0805 -> Capacitors_SMD:C_0603
- R1: value 1K -> 10K
Connections:
- net TX: now also P1.7 (P7); no longer P1.5 (P5)
- net at P1.4 (P4): no longer R2.2
- net at P1.8 (P8): now also R2.2
Changed lines of the file:
@@
 $EndComp
 $Comp
-L GND #PWR10
+L GND #PWR01
 U 1 1 58A7255A
 P 6200 3700
-F 0 "#PWR10" H 6200 3450 50  0001 C CNN
+F 0 "#PWR01" H 6200 3450 50  0001 C CNN
 F 1 "GND" H 6200 3550 50  0000 C CNN
 F 2 "" H 6200 3700 50  0000 C CNN
@@
 Connection ~ 6200 3250
 $Comp
-L +5V #PWR5
+L +5V #PWR02
 U 1 1 58A725A3
 P 4600 2600
-F 0 "#PWR5" H 4600 2450 50  0001 C CNN
+F 0 "#PWR02" H 4600 2450 50  0001 C CNN
 F 1 "+5V" H 4600 2740 50  0000 C CNN
 F 2 "" H 4600 2600 50  0000 C CNN
@@
 $EndComp
 $Comp
-L +5V #PWR4
+L +5V #PWR03
 U 1 1 58A725D3
 P 3850 1150
-F 0 "#PWR4" H 3850 1000 50  0001 C CNN
+F 0 "#PWR03" H 3850 1000 50  0001 C CNN
 F 1 "+5V" H 3850 1290 50  0000 C CNN
 F 2 "" H 3850 1150 50  0000 C CNN
@@
 $EndComp
 $Comp
-L GND #PWR9
+L GND #PWR04
 U 1 1 58A7262B
 P 6150 1650
-F 0 "#PWR9" H 6150 1400 50  0001 C CNN
+F 0 "#PWR04" H 6150 1400 50  0001 C CNN
 F 1 "GND" H 6150 1500 50  0000 C CNN
 F 2 "" H 6150 1650 50  0000 C CNN
@@
 F 0 "C2" H 4375 1500 50  0000 L CNN
 F 1 "10nF" H 4375 1300 50  0000 L CNN
-F 2 "Capacitors_SMD:C_0805" H 4050 1100 50  0000 C CNN
+F 2 "Capacitors_SMD:C_0603" H 4050 1100 50  0000 C CNN
 F 3 "" H 4350 1400 50  0000 C CNN
 	1    4350 1400
@@
 F 0 "C3" H 7075 3350 50  0000 L CNN
 F 1 "10nF" H 7075 3150 50  0000 L CNN
-F 2 "Capacitors_SMD:C_0805" V 7300 3150 50  0000 C CNN
+F 2 "Capacitors_SMD:C_0603" V 7300 3150 50  0000 C CNN
 F 3 "" H 7050 3250 50  0000 C CNN
 	1    7050 3250
@@
 F 0 "C4" H 7525 3350 50  0000 L CNN
 F 1 "10nF" H 7525 3150 50  0000 L CNN
-F 2 "Capacitors_SMD:C_0805" V 7750 3450 50  0000 C CNN
+F 2 "Capacitors_SMD:C_0603" V 7750 3450 50  0000 C CNN
 F 3 "" H 7500 3250 50  0000 C CNN
 	1    7500 3250
@@
 F 0 "C1" H 4025 3000 50  0000 L CNN
 F 1 "10nF" H 4025 2800 50  0000 L CNN
-F 2 "Capacitors_SMD:C_0805" V 4250 3150 50  0000 C CNN
+F 2 "Capacitors_SMD:C_0603" V 4250 3150 50  0000 C CNN
 F 3 "" H 4000 2900 50  0000 C CNN
 	1    4000 2900
@@
 P 4600 3500
 F 0 "R1" V 4680 3500 50  0000 C CNN
-F 1 "1K" V 4600 3500 50  0000 C CNN
+F 1 "10K" V 4600 3500 50  0000 C CNN
 F 2 "Resistors_SMD:R_0603" V 4450 3400 50  0000 C CNN
 F 3 "" H 4600 3500 50  0000 C CNN
@@
 $EndComp
 $Comp
-L GND #PWR6
+L GND #PWR05
 U 1 1 58A72FF9
 P 4600 3800
-F 0 "#PWR6" H 4600 3550 50  0001 C CNN
+F 0 "#PWR05" H 4600 3550 50  0001 C CNN
 F 1 "GND" H 4600 3650 50  0000 C CNN
 F 2 "" H 4600 3800 50  0000 C CNN
@@
 $EndComp
 $Comp
-L GND #PWR1
+L GND #PWR06
 U 1 1 58A73EAE
 P 2800 5450
-F 0 "#PWR1" H 2800 5200 50  0001 C CNN
+F 0 "#PWR06" H 2800 5200 50  0001 C CNN
 F 1 "GND" H 2800 5300 50  0000 C CNN
 F 2 "" H 2800 5450 50  0000 C CNN
@@
 $EndComp
 $Comp
-L +5V #PWR2
+L +5V #PWR07
 U 1 1 58A73ED7
 P 3200 5100
-F 0 "#PWR2" H 3200 4950 50  0001 C CNN
+F 0 "#PWR07" H 3200 4950 50  0001 C CNN
 F 1 "+5V" H 3200 5240 50  0000 C CNN
 F 2 "" H 3200 5100 50  0000 C CNN
@@
 Text GLabel 2650 4800 2    47   Output ~ 0
 ANT_SWITCH
-Wire Wire Line
-	3200 5000 2450 5000
 Text GLabel 3850 2600 0    47   BiDi ~ 0
 ANT
@@
 Text GLabel 8000 3800 2    47   BiDi ~ 0
 ANT_RX
-Text GLabel 2650 4900 2    47   Output ~ 0
+Text GLabel 2650 4700 2    47   Output ~ 0
 TX
 Text GLabel 3650 4100 2    47   Input ~ 0
 RX
-Wire Wire Line
-	2450 4900 2650 4900
 $Comp
 L CONN_01X04 P2
@@
 $EndComp
 $Comp
-L +5V #PWR7
+L +5V #PWR08
 U 1 1 58A74262
 P 5250 4550
-F 0 "#PWR7" H 5250 4400 50  0001 C CNN
+F 0 "#PWR08" H 5250 4400 50  0001 C CNN
 F 1 "+5V" H 5250 4690 50  0000 C CNN
 F 2 "" H 5250 4550 50  0000 C CNN
@@
 $EndComp
 $Comp
-L +5V #PWR12
+L +5V #PWR09
 U 1 1 58A74294
 P 7600 4200
-F 0 "#PWR12" H 7600 4050 50  0001 C CNN
+F 0 "#PWR09" H 7600 4050 50  0001 C CNN
 F 1 "+5V" H 7600 4340 50  0000 C CNN
 F 2 "" H 7600 4200 50  0000 C CNN
@@
 $EndComp
 $Comp
-L +5V #PWR13
+L +5V #PWR010
 U 1 1 58A742C6
 P 7600 4900
-F 0 "#PWR13" H 7600 4750 50  0001 C CNN
+F 0 "#PWR010" H 7600 4750 50  0001 C CNN
 F 1 "+5V" H 7600 5040 50  0000 C CNN
 F 2 "" H 7600 4900 50  0000 C CNN
@@
 $EndComp
 $Comp
-L GND #PWR8
+L GND #PWR011
 U 1 1 58A742F8
 P 5300 5200
-F 0 "#PWR8" H 5300 4950 50  0001 C CNN
+F 0 "#PWR011" H 5300 4950 50  0001 C CNN
 F 1 "GND" H 5300 5050 50  0000 C CNN
 F 2 "" H 5300 5200 50  0000 C CNN
@@
 $EndComp
 $Comp
-L GND #PWR14
+L GND #PWR012
 U 1 1 58A7432A
 P 7600 5550
-F 0 "#PWR14" H 7600 5300 50  0001 C CNN
+F 0 "#PWR012" H 7600 5300 50  0001 C CNN
 F 1 "GND" H 7600 5400 50  0000 C CNN
 F 2 "" H 7600 5550 50  0000 C CNN
@@
 	7500 4350 7500 4400
 $Comp
-L GND #PWR11
+L GND #PWR013
 U 1 1 58A74736
 P 7500 4400
-F 0 "#PWR11" H 7500 4150 50  0001 C CNN
+F 0 "#PWR013" H 7500 4150 50  0001 C CNN
 F 1 "GND" H 7500 4250 50  0000 C CNN
 F 2 "" H 7500 4400 50  0000 C CNN
@@
 $EndComp
 $Comp
-L GND #PWR15
+L GND #PWR014
 U 1 1 58A76A15
 P 8100 1950
-F 0 "#PWR15" H 8100 1700 50  0001 C CNN
+F 0 "#PWR014" H 8100 1700 50  0001 C CNN
 F 1 "GND" H 8100 1800 50  0000 C CNN
 F 2 "" H 8100 1950 50  0000 C CNN
@@
 $EndComp
 Wire Wire Line
-	3200 4500 3200 5000
-Wire Wire Line
 	3200 4200 3200 4100
 $Comp
@@
 $EndComp
 $Comp
-L GND #PWR3
+L GND #PWR015
 U 1 1 58A78CFD
 P 3450 4600
-F 0 "#PWR3" H 3450 4350 50  0001 C CNN
+F 0 "#PWR015" H 3450 4350 50  0001 C CNN
 F 1 "GND" H 3450 4450 50  0000 C CNN
 F 2 "" H 3450 4600 50  0000 C CNN
@@
 Wire Wire Line
 	2450 4800 2650 4800
+Wire Wire Line
+	2450 4600 3200 4600
+Wire Wire Line
+	3200 4600 3200 4500
+Wire Wire Line
+	2450 4700 2650 4700
 $EndSCHEMATC
